File: PCB/IoT_Devices_Blink/IoT_Devices_Blink.kicad_sch (KiCad schematic)
At the start: 6 parts, among them J1 Conn_01x07_Socket, J2 Conn_01x07_Socket, SW1 SW_Push

Commit message: Create basic blink iot dashboard
Parts:
- J1, J2: footprint Connector_PinHeader_2.54mm:PinHeader_1x07_P2.54mm_Vertical -> Connector_PinSocket_2.54mm:PinSocket_1x07_P2.54mm_Vertical
Changed lines of the file:
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@@
 		)
 		(instances
-			(project ""
+			(project "IoT_Devices_Blink"
 				(path "/b5283d16-bf3a-4bc2-be4d-4f67771ecd29"
 					(reference "D1")
@@
 		)
 		(instances
-			(project ""
+			(project "IoT_Devices_Blink"
 				(path "/b5283d16-bf3a-4bc2-be4d-4f67771ecd29"
 					(reference "C1")
@@
 		)
 		(instances
-			(project ""
+			(project "IoT_Devices_Blink"
 				(path "/b5283d16-bf3a-4bc2-be4d-4f67771ecd29"
 					(reference "SW1")
@@
 		)
 		(instances
-			(project "Blink"
+			(project "IoT_Devices_Blink"
 				(path "/b5283d16-bf3a-4bc2-be4d-4f67771ecd29"
 					(reference "R1")
@@
 			)
 		)
-		(property "Footprint" "Connector_PinHeader_2.54mm:PinHeader_1x07_P2.54mm_Vertical"
+		(property "Footprint" "Connector_PinSocket_2.54mm:PinSocket_1x07_P2.54mm_Vertical"
 			(at 85.09 59.69 0)
 			(effects
@@
 		)
 		(instances
-			(project ""
+			(project "IoT_Devices_Blink"
 				(path "/b5283d16-bf3a-4bc2-be4d-4f67771ecd29"
 					(reference "J1")
@@
 			)
 		)
-		(property "Footprint" "Connector_PinHeader_2.54mm:PinHeader_1x07_P2.54mm_Vertical"
+		(property "Footprint" "Connector_PinSocket_2.54mm:PinSocket_1x07_P2.54mm_Vertical"
 			(at 93.98 59.69 0)
 			(effects
@@
 		)
 		(instances
-			(project "Blink"
+			(project "IoT_Devices_Blink"
 				(path "/b5283d16-bf3a-4bc2-be4d-4f67771ecd29"
 					(reference "J2")
